File: hardware/programator.kicad_sch (KiCad schematic)
At the start: 1 part, among them J2 FTSH-107-01-L-DV-K-A

Commit message: connectors - added, buses - todo
Connections:
- net +3.3V renamed +3V3
Changed lines of the file:
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@@
+		)
+	)
+	(bus
+		(pts
+			(xy 165.735 95.25) (xy 169.545 95.25)
+		)
+		(stroke
+			(width 0)
+			(type default)
+		)
+	)
+	(wire
+		(pts
+			(xy 163.195 107.95) (xy 163.195 110.49)
+		)
+		(stroke
+			(width 0)
+			(type default)
+		)
+	)
+	(wire
+		(pts
+			(xy 155.575 100.33) (xy 163.195 100.33)
+		)
+		(stroke
+			(width 0)
+			(type default)
 		)
 	)
@@
 		(pts
 			(xy 155.575 110.49) (xy 163.195 110.49)
-		)
-		(stroke
-			(width 0)
-			(type default)
-		)
-	)
-	(bus
-		(pts
-			(xy 165.735 95.25) (xy 169.545 95.25)
-		)
-		(stroke
-			(width 0)
-			(type default)
-		)
-	)
-	(wire
-		(pts
-			(xy 155.575 100.33) (xy 163.195 100.33)
 		)
 		(stroke
@@
 		)
 	)
-	(label "RST"
-		(at 163.195 110.49 180)
-		(fields_autoplaced yes)
-		(effects
-			(font
-				(size 1.27 1.27)
-			)
-			(justify right bottom)
+	(global_label "RST"
+		(shape input)
+		(at 163.195 107.95 0)
+		(fields_autoplaced yes)
+		(effects
+			(font
+				(size 1.27 1.27)
+			)
+			(justify left)
+		)
+		(property "Intersheetrefs" "${INTERSHEET_REFS}"
+			(at 169.6273 107.95 0)
+			(effects
+				(font
+					(size 1.27 1.27)
+				)
+				(justify left)
+				(hide yes)
+			)
 		)
 	)
@@
 	)
 	(symbol
-		(lib_id "power:+3.3V")
+		(lib_id "power:+3V3")
 		(at 125.095 99.06 0)
 		(unit 1)
@@
 			)
 		)
-		(property "Value" "+3.3V"
+		(property "Value" "+3V3"
 			(at 125.095 93.98 0)
 			(effects
@@
 			)
 		)
-		(property "Description" ""
+		(property "Description" "Power symbol creates a global label with name \"+3V3\""
 			(at 125.095 99.06 0)
 			(effects

Commit message: Poprawione busy, brak errorow
Changed lines of the file:
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@@
 	(paper "A4")
 	(junction
-		(at 125.095 105.41)
+		(at 118.11 105.41)
 		(diameter 0)
 		(color 0 0 0 0)
 	)
 	(junction
-		(at 125.095 110.49)
+		(at 118.11 110.49)
 		(diameter 0)
 		(color 0 0 0 0)
@@
 	(no_connect
 		(at 155.575 107.95)
+	)
+	(bus_entry
+		(at 121.92 113.03)
+		(size -2.54 2.54)
+		(stroke
+			(width 0)
+			(type default)
+		)
 	)
 	(bus_entry
@@
 	)
 	(bus_entry
-		(at 166.37 117.475)
-		(size 2.54 -2.54)
-		(stroke
-			(width 0)
-			(type default)
-		)
-	)
-	(bus_entry
 		(at 163.195 100.33)
 		(size 2.54 -2.54)
@@
 		)
 	)
-	(wire
-		(pts
-			(xy 131.445 113.03) (xy 131.445 117.475)
-		)
-		(stroke
-			(width 0)
-			(type default)
-		)
-	)
-	(wire
-		(pts
-			(xy 125.095 100.33) (xy 132.715 100.33)
+	(bus
+		(pts
+			(xy 115.57 114.935) (xy 119.38 114.935)
+		)
+		(stroke
+			(width 0)
+			(type default)
+		)
+	)
+	(bus
+		(pts
+			(xy 119.38 115.57) (xy 119.38 114.935)
+		)
+		(stroke
+			(width 0)
+			(type default)
+		)
+	)
+	(wire
+		(pts
+			(xy 118.11 100.33) (xy 132.715 100.33)
 		)
 		(stroke
@@
 	(wire
 		(pts
-			(xy 125.095 111.76) (xy 125.095 110.49)
+			(xy 117.475 110.49) (xy 118.11 110.49)
 		)
 		(stroke
@@
 	(wire
 		(pts
-			(xy 131.445 113.03) (xy 132.715 113.03)
-		)
-		(stroke
-			(width 0)
-			(type default)
-		)
-	)
-	(wire
-		(pts
-			(xy 125.095 105.41) (xy 125.095 102.87)
+			(xy 121.92 113.03) (xy 132.715 113.03)
+		)
+		(stroke
+			(width 0)
+			(type default)
+		)
+	)
+	(wire
+		(pts
+			(xy 118.11 105.41) (xy 118.11 102.87)
 		)
 		(stroke
@@
 	(wire
 		(pts
-			(xy 125.095 110.49) (xy 132.715 110.49)
-		)
-		(stroke
-			(width 0)
-			(type default)
-		)
-	)
-	(wire
-		(pts
-			(xy 166.37 117.475) (xy 131.445 117.475)
-		)
-		(stroke
-			(width 0)
-			(type default)
-		)
-	)
-	(bus
-		(pts
-			(xy 168.91 110.49) (xy 168.91 114.935)
-		)
-		(stroke
-			(width 0)
-			(type default)
-		)
-	)
-	(wire
-		(pts
-			(xy 125.095 102.87) (xy 132.715 102.87)
-		)
-		(stroke
-			(width 0)
-			(type default)
-		)
-	)
-	(wire
-		(pts
-			(xy 125.095 99.06) (xy 125.095 100.33)
-		)
-		(stroke
-			(width 0)
-			(type default)
-		)
-	)
-	(wire
-		(pts
-			(xy 125.095 105.41) (xy 125.095 110.49)
+			(xy 118.11 110.49) (xy 132.715 110.49)
+		)
+		(stroke
+			(width 0)
+			(type default)
+		)
+	)
+	(wire
+		(pts
+			(xy 118.11 102.87) (xy 132.715 102.87)
+		)
+		(stroke
+			(width 0)
+			(type default)
+		)
+	)
+	(wire
+		(pts
+			(xy 118.11 99.06) (xy 118.11 100.33)
+		)
+		(stroke
+			(width 0)
+			(type default)
+		)
+	)
+	(wire
+		(pts
+			(xy 118.11 105.41) (xy 118.11 110.49)
 		)
 		(stroke
@@
 	(wire
 		(pts
-			(xy 125.095 105.41) (xy 132.715 105.41)
+			(xy 118.11 105.41) (xy 132.715 105.41)
 		)
 		(stroke
@@
 	)
 	(rectangle
-		(start 113.665 85.09)
+		(start 98.425 85.09)
 		(end 191.135 128.27)
 		(stroke
@@
 	(text "PROGRAMATOR"
 		(exclude_from_sim no)
-		(at 113.665 83.185 0)
+		(at 98.425 83.185 0)
 		(effects
 			(font
@@
 		)
 	)
-	(label "USART1_RX"
-		(at 166.37 117.475 180)
-		(fields_autoplaced yes)
-		(effects
-			(font
-				(size 1.27 1.27)
-			)
-			(justify right bottom)
-		)
-	)
 	(label "SWDIO"
 		(at 163.195 100.33 180)
+		(fields_autoplaced yes)
+		(effects
+			(font
+				(size 1.27 1.27)
+			)
+			(justify right bottom)
+		)
+	)
+	(label "USART1_RX"
+		(at 132.715 113.03 180)
 		(fields_autoplaced yes)
 		(effects
@@
 		)
 	)
+	(hierarchical_label "USART1{TX RX}"
+		(shape bidirectional)
+		(at 115.57 114.935 180)
+		(fields_autoplaced yes)
+		(effects
+			(font
+				(size 1.27 1.27)
+			)
+			(justify right)
+		)
+	)
 	(hierarchical_label "SW{SWDIO SWCLK}"
 		(shape input)
@@
 	(symbol
 		(lib_id "power:GND")
-		(at 125.095 111.76 0)
-		(mirror y)
+		(at 117.475 110.49 270)
+		(mirror x)
 		(unit 1)
 		(exclude_from_sim no)
@@
 		(dnp no)
 		(property "Reference" "#PWR010"
-			(at 125.095 118.11 0)
+			(at 111.125 110.49 0)
 			(effects
 				(font
@@
 		)
 		(property "Value" "GND"
-			(at 125.095 116.84 0)
+			(at 112.395 110.49 0)
 			(effects
 				(font
@@
 		)
 		(property "Footprint" ""
-			(at 125.095 111.76 0)
+			(at 117.475 110.49 0)
 			(effects
 				(font
@@
 		)
 		(property "Datasheet" ""
-			(at 125.095 111.76 0)
+			(at 117.475 110.49 0)
 			(effects
 				(font
@@
 		)
 		(property "Description" ""
-			(at 125.095 111.76 0)
+			(at 117.475 110.49 0)
 			(effects
 				(font
@@
 	(symbol
 		(lib_id "power:+3V3")
-		(at 125.095 99.06 0)
+		(at 118.11 99.06 0)
 		(unit 1)
 		(exclude_from_sim no)
@@
 		(fields_autoplaced yes)
 		(property "Reference" "#PWR09"
-			(at 125.095 102.87 0)
+			(at 118.11 102.87 0)
 			(effects
 				(font
@@
 		)
 		(property "Value" "+3V3"
-			(at 125.095 93.98 0)
+			(at 118.11 93.98 0)
 			(effects
 				(font
@@
 		)
 		(property "Footprint" ""
-			(at 125.095 99.06 0)
+			(at 118.11 99.06 0)
 			(effects
 				(font
@@
 		)
 		(property "Datasheet" ""
-			(at 125.095 99.06 0)
+			(at 118.11 99.06 0)
 			(effects
 				(font
@@
 		)
 		(property "Description" "Power symbol creates a global label with name \"+3V3\""
-			(at 125.095 99.06 0)
-			(effects
-				(font
+			(at 118.11 99.06 0)
+			(effects
+				(font
