File: hardware/_autosave-power.kicad_sch (KiCad schematic)
At the start: 61 parts, among them IC1 LMR38020FDDAR, Q1 LMR51635XDDCR, Q2 LMR51635XDDCR, T1 TP_VCC, T10 TP_+3V3, T11 TP_+5V, T12 TP_+5V, T2 TP_VCC, T3 TP_VCC, T4 TP_VCC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

Commit message: nowy uklad
Parts:
- F4: footprint SamacSys_Parts:MINIASMDC260F162 -> Fuse:Fuse_1812_4532Metric_Pad1.30x3.40mm_HandSolder
Changed lines of the file:
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@@
 			)
 		)
-		(property "Footprint" "SamacSys_Parts:MINIASMDC260F162"
+		(property "Footprint" "Fuse:Fuse_1812_4532Metric_Pad1.30x3.40mm_HandSolder"
 			(at 231.14 114.3 0)
 			(effects
