File: hardware/can.kicad_sch (KiCad schematic)
At the start: 10 parts, among them U3 MCP2542FDxMF

Commit message: Items assebled
Parts:
- renumbered TP14 to T14, TP15 to T15, TP16 to T16, TP17 to T17
Changed lines of the file:
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@@
 		(dnp no)
 		(fields_autoplaced yes)
-		(property "Reference" "TP17"
+		(property "Reference" "T17"
 			(at 201.93 116.8399 0)
 			(effects
@@
 			(project "drs"
 				(path "/b652b05a-4e3d-4ad1-b032-18886abe7d45/b1fd2a01-bf35-4031-ba71-28db4e5321a0"
-					(reference "TP17")
+					(reference "T17")
 					(unit 1)
 				)
@@
 		(on_board yes)
 		(dnp no)
-		(property "Reference" "TP14"
+		(property "Reference" "T14"
 			(at 102.87 85.0899 0)
 			(effects
@@
 			(project "drs"
 				(path "/b652b05a-4e3d-4ad1-b032-18886abe7d45/b1fd2a01-bf35-4031-ba71-28db4e5321a0"
-					(reference "TP14")
+					(reference "T14")
 					(unit 1)
 				)
@@
 		(dnp no)
 		(fields_autoplaced yes)
-		(property "Reference" "TP15"
+		(property "Reference" "T15"
 			(at 130.81 85.0899 0)
 			(effects
@@
 			(project "drs"
 				(path "/b652b05a-4e3d-4ad1-b032-18886abe7d45/b1fd2a01-bf35-4031-ba71-28db4e5321a0"
-					(reference "TP15")
+					(reference "T15")
 					(unit 1)
 				)
@@
 		(dnp no)
 		(fields_autoplaced yes)
-		(property "Reference" "TP16"
+		(property "Reference" "T16"
 			(at 201.93 91.4399 0)
 			(effects
@@
 			(project "drs"
 				(path "/b652b05a-4e3d-4ad1-b032-18886abe7d45/b1fd2a01-bf35-4031-ba71-28db4e5321a0"
-					(reference "TP16")
-					(unit 1)
-				)
+					(reference "T16")
+					(unit 1)
+				)

Commit message: schematic & pcb update
Parts:
- renumbered D4 to D8, R14 to R17, T14 to T13, T15 to T14, T16 to T15, T17 to T16
Changed lines of the file:
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@@
 		(dnp no)
 		(fields_autoplaced yes)
-		(property "Reference" "#PWR0138"
+		(property "Reference" "#PWR037"
 			(at 104.14 127 0)
 			(effects
@@
 			(project "drs"
 				(path "/b652b05a-4e3d-4ad1-b032-18886abe7d45/b1fd2a01-bf35-4031-ba71-28db4e5321a0"
-					(reference "#PWR0138")
+					(reference "#PWR037")
 					(unit 1)
 				)
@@
 		(dnp no)
 		(fields_autoplaced yes)
-		(property "Reference" "R14"
+		(property "Reference" "R17"
 			(at 177.8 109.2199 0)
 			(effects
@@
 			(project "drs"
 				(path "/b652b05a-4e3d-4ad1-b032-18886abe7d45/b1fd2a01-bf35-4031-ba71-28db4e5321a0"
-					(reference "R14")
+					(reference "R17")
 					(unit 1)
 				)
@@
 		(dnp no)
 		(fields_autoplaced yes)
-		(property "Reference" "#PWR0136"
+		(property "Reference" "#PWR035"
 			(at 104.14 86.36 0)
 			(effects
@@
 			(project "drs"
 				(path "/b652b05a-4e3d-4ad1-b032-18886abe7d45/b1fd2a01-bf35-4031-ba71-28db4e5321a0"
-					(reference "#PWR0136")
+					(reference "#PWR035")
 					(unit 1)
 				)
@@
 		(dnp no)
 		(fields_autoplaced yes)
-		(property "Reference" "#PWR0137"
+		(property "Reference" "#PWR038"
 			(at 118.11 132.08 0)
 			(effects
@@
 			(project "drs"
 				(path "/b652b05a-4e3d-4ad1-b032-18886abe7d45/b1fd2a01-bf35-4031-ba71-28db4e5321a0"
-					(reference "#PWR0137")
+					(reference "#PWR038")
 					(unit 1)
 				)
@@
 		(dnp no)
 		(fields_autoplaced yes)
-		(property "Reference" "T17"
+		(property "Reference" "T16"
 			(at 201.93 116.8399 0)
 			(effects
@@
 			(project "drs"
 				(path "/b652b05a-4e3d-4ad1-b032-18886abe7d45/b1fd2a01-bf35-4031-ba71-28db4e5321a0"
-					(reference "T17")
+					(reference "T16")
 					(unit 1)
 				)
@@
 		(on_board yes)
 		(dnp no)
-		(property "Reference" "T14"
+		(property "Reference" "T13"
 			(at 102.87 85.0899 0)
 			(effects
@@
 			(project "drs"
 				(path "/b652b05a-4e3d-4ad1-b032-18886abe7d45/b1fd2a01-bf35-4031-ba71-28db4e5321a0"
-					(reference "T14")
+					(reference "T13")
 					(unit 1)
 				)
@@
 		(dnp no)
 		(fields_autoplaced yes)
-		(property "Reference" "#PWR0133"
+		(property "Reference" "#PWR040"
 			(at 129.54 102.87 0)
 			(effects
@@
 			(project "drs"
 				(path "/b652b05a-4e3d-4ad1-b032-18886abe7d45/b1fd2a01-bf35-4031-ba71-28db4e5321a0"
-					(reference "#PWR0133")
+					(reference "#PWR040")
 					(unit 1)
 				)
@@
 		(dnp no)
 		(fields_autoplaced yes)
-		(property "Reference" "T15"
+		(property "Reference" "T14"
 			(at 130.81 85.0899 0)
 			(effects
@@
 			(project "drs"
 				(path "/b652b05a-4e3d-4ad1-b032-18886abe7d45/b1fd2a01-bf35-4031-ba71-28db4e5321a0"
-					(reference "T15")
+					(reference "T14")
 					(unit 1)
 				)
@@
 		(dnp no)
 		(fields_autoplaced yes)
-		(property "Reference" "T16"
+		(property "Reference" "T15"
 			(at 201.93 91.4399 0)
 			(effects
@@
 			(project "drs"
 				(path "/b652b05a-4e3d-4ad1-b032-18886abe7d45/b1fd2a01-bf35-4031-ba71-28db4e5321a0"
-					(reference "T16")
+					(reference "T15")
 					(unit 1)
 				)
@@
 		(on_board yes)
 		(dnp no)
-		(property "Reference" "D4"
+		(property "Reference" "D8"
 			(at 194.31 106.68 0)
 			(effects
@@
 			(project "drs"
 				(path "/b652b05a-4e3d-4ad1-b032-18886abe7d45/b1fd2a01-bf35-4031-ba71-28db4e5321a0"
-					(reference "D4")
+					(reference "D8")
 					(unit 1)
 				)
@@
 		(dnp no)
 		(fields_autoplaced yes)
-		(property "Reference" "#PWR0134"
+		(property "Reference" "#PWR039"
 			(at 129.54 86.36 0)
 			(effects
@@
 			(project "drs"
 				(path "/b652b05a-4e3d-4ad1-b032-18886abe7d45/b1fd2a01-bf35-4031-ba71-28db4e5321a0"
-					(reference "#PWR0134")
+					(reference "#PWR039")
 					(unit 1)
 				)
@@
 		(dnp no)
 		(fields_autoplaced yes)
-		(property "Reference" "#PWR0135"
+		(property "Reference" "#PWR036"
 			(at 104.14 102.87 0)
 			(effects
@@
 			(project "drs"
 				(path "/b652b05a-4e3d-4ad1-b032-18886abe7d45/b1fd2a01-bf35-4031-ba71-28db4e5321a0"
-					(reference "#PWR0135")
+					(reference "#PWR036")
 					(unit 1)
 				)
@@
 		(dnp no)
 		(fields_autoplaced yes)
-		(property "Reference" "#PWR0132"
+		(property "Reference" "#PWR041"
 			(at 207.01 114.3 0)
 			(effects
@@
 			(project "drs"
 				(path "/b652b05a-4e3d-4ad1-b032-18886abe7d45/b1fd2a01-bf35-4031-ba71-28db4e5321a0"
-					(reference "#PWR0132")
-					(unit 1)
-				)
+					(reference "#PWR041")
+					(unit 1)
+				)
