File: hardware/can.kicad_sch (KiCad schematic)
At the start: 10 parts, among them T13 TP_+3V3, T14 TP_+5V, T15 TP_CAN_H, T16 TP_CAN_L, U3 MCP2542FDxMF

Commit message: pcb update
Connections:
- net CAN_H renamed CAN_P
- net CAN_L renamed CAN_N
Changed lines of the file:
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@@
 		)
 	)
-	(hierarchical_label "CAN_L"
+	(hierarchical_label "CAN_N"
 		(shape bidirectional)
 		(at 130.81 116.84 0)
@@
 		)
 	)
-	(hierarchical_label "CAN_H"
+	(hierarchical_label "CAN_P"
 		(shape bidirectional)
 		(at 130.81 111.76 0)
@@
 		)
 	)
-	(hierarchical_label "CAN_L"
+	(hierarchical_label "CAN_N"
 		(shape bidirectional)
 		(at 158.75 118.11 180)
@@
 		)
 	)
-	(hierarchical_label "CAN_H"
+	(hierarchical_label "CAN_P"
 		(shape bidirectional)
 		(at 158.75 92.71 180)

Commit message: Added author on pcb
Other:
- company: (none) -> Author: Grzegorz Potocki
- title: (none) -> DRS - Drag Reduction System
Changed lines of the file:
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@@
 	(generator_version "9.0")
 	(paper "A4")
+	(title_block
+		(title "DRS - Drag Reduction System")
+		(date "2024-11-28")
+		(rev "${REVISION}")
+		(company "Author: Grzegorz Potocki")
+		(comment 1 "Reviewer: Jakub Drankiewicz")
+	)
 	(rectangle
 		(start 73.66 69.85)
