File: hardware/control.kicad_sch (KiCad schematic)
At the start: 8 parts, among them U1 STM32G0C1KCTxN

Commit message: pcb scheme update - general/basic aligment
Parts:
- renumbered C6 to C1, C1 to C2, C2 to C3, C3 to C4, C4 to C5, R4 to R2
Changed lines of the file:
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@@
 (kicad_sch
-	(version 20231120)
+	(version 20250114)
 	(generator "eeschema")
-	(generator_version "8.0")
+	(generator_version "9.0")
 	(paper "A4")
 	(bus_alias "CAN"
@@
 	(bus_alias "USB"
 		(members "D-" "D+")
+	)
+	(rectangle
+		(start 62.865 44.45)
+		(end 222.25 158.115)
+		(stroke
+			(width 0)
+			(type default)
+		)
+		(fill
+			(type none)
+		)
+	)
+	(text "STM32"
+		(exclude_from_sim no)
+		(at 63.5 43.18 0)
+		(effects
+			(font
+				(size 3 3)
+				(thickness 2)
+				(bold yes)
+				(italic yes)
+			)
+			(justify left)
+		)
 	)
 	(junction
@@
 		)
 	)
-	(rectangle
-		(start 62.865 44.45)
-		(end 222.25 158.115)
-		(stroke
-			(width 0)
-			(type default)
-		)
-		(fill
-			(type none)
-		)
-	)
-	(text "STM32"
-		(exclude_from_sim no)
-		(at 63.5 43.18 0)
-		(effects
-			(font
-				(size 3 3)
-				(thickness 2)
-				(bold yes)
-				(italic yes)
-			)
-			(justify left)
-		)
-	)
 	(label "TXD"
 		(at 125.73 91.44 0)
-		(fields_autoplaced yes)
 		(effects
 			(font
@@
 	(label "{USART1}"
 		(at 113.03 109.22 0)
-		(fields_autoplaced yes)
 		(effects
 			(font
@@
 	(label "LED_WRN"
 		(at 124.46 101.6 0)
-		(fields_autoplaced yes)
 		(effects
 			(font
@@
 	(label "TX"
 		(at 124.46 114.3 0)
-		(fields_autoplaced yes)
 		(effects
 			(font
@@
 	(label "CLK"
 		(at 173.99 119.38 0)
-		(fields_autoplaced yes)
 		(effects
 			(font
@@
 	(label "LED_ERR"
 		(at 124.46 121.92 0)
-		(fields_autoplaced yes)
 		(effects
 			(font
@@
 	(label "{USB}"
 		(at 196.85 106.68 180)
-		(fields_autoplaced yes)
 		(effects
 			(font
@@
 	(label "PWM1"
 		(at 185.42 86.36 180)
-		(fields_autoplaced yes)
 		(effects
 			(font
@@
 	(label "D-"
 		(at 173.99 111.76 0)
-		(fields_autoplaced yes)
 		(effects
 			(font
@@
 	(label "MOSI"
 		(at 185.42 93.98 180)
-		(fields_autoplaced yes)
 		(effects
 			(font
@@
 	(label "PWM2"
 		(at 185.42 88.9 180)
-		(fields_autoplaced yes)
 		(effects
 			(font
@@
 	(label "{SW}"
 		(at 198.12 116.84 180)
-		(fields_autoplaced yes)
 		(effects
 			(font
@@
 	(label "LED_OK"
 		(at 124.46 119.38 0)
-		(fields_autoplaced yes)
 		(effects
 			(font
@@
 	(label "RX"
 		(at 124.46 116.84 0)
-		(fields_autoplaced yes)
 		(effects
 			(font
@@
 	(label "D+"
 		(at 173.99 114.3 0)
-		(fields_autoplaced yes)
 		(effects
 			(font
@@
 	(label "STM_VCC"
 		(at 156.21 55.88 180)
-		(fields_autoplaced yes)
 		(effects
 			(font
@@
 	(label "{PWM}"
 		(at 204.47 86.36 180)
-		(fields_autoplaced yes)
 		(effects
 			(font
@@
 	(label "RXD"
 		(at 125.73 88.9 0)
-		(fields_autoplaced yes)
 		(effects
 			(font
@@
 	(label "{CAN}"
 		(at 114.3 88.9 0)
-		(fields_autoplaced yes)
 		(effects
 			(font
@@
 	(label "{SPI}"
 		(at 198.12 78.74 180)
-		(fields_autoplaced yes)
 		(effects
 			(font
@@
 	(label "NRST"
 		(at 130.81 83.82 0)
-		(fields_autoplaced yes)
 		(effects
 			(font
@@
 	(label "DIO"
 		(at 173.99 116.84 0)
-		(fields_autoplaced yes)
 		(effects
 			(font
@@
 	(label "SCK"
 		(at 185.42 83.82 180)
-		(fields_autoplaced yes)
 		(effects
 			(font
@@
 	(label "MISO"
 		(at 185.42 91.44 180)
-		(fields_autoplaced yes)
 		(effects
 			(font
@@
 			)
 			(justify right bottom)
-		)
-	)
-	(global_label "RST"
-		(shape input)
-		(at 121.92 80.01 0)
-		(fields_autoplaced yes)
-		(effects
-			(font
-				(size 1.27 1.27)
-			)
-			(justify left)
-		)
-		(property "Intersheetrefs" "${INTERSHEET_REFS}"
-			(at 128.3523 80.01 0)
-			(effects
-				(font
-					(size 1.27 1.27)
-				)
-				(justify left)
-				(hide yes)
-			)
 		)
 	)
@@
 		(shape bidirectional)
 		(at 198.12 78.74 0)
-		(fields_autoplaced yes)
 		(effects
 			(font
@@
 		(shape output)
 		(at 204.47 86.36 0)
-		(fields_autoplaced yes)
+		(effects
+			(font
+				(size 1.27 1.27)
+			)
+			(justify left)
+		)
+	)
+	(hierarchical_label "RST"
+		(shape input)
+		(at 121.92 80.01 0)
 		(effects
 			(font
@@
 		(shape bidirectional)
 		(at 198.12 116.84 0)
-		(fields_autoplaced yes)
 		(effects
 			(font
@@
 		(shape bidirectional)
 		(at 114.3 88.9 180)
-		(fields_autoplaced yes)
 		(effects
 			(font
@@
 		(shape output)
 		(at 198.12 106.68 0)
-		(fields_autoplaced yes)
 		(effects
 			(font
@@
 		(shape bidirectional)
 		(at 113.03 109.22 180)
-		(fields_autoplaced yes)
 		(effects
 			(font
@@
 		(dnp no)
 		(fields_autoplaced yes)
-		(property "Reference" "#PWR029"
+		(property "Reference" "#PWR0102"
 			(at 71.12 57.15 0)
 			(effects
@@
 			(project "drs"
 				(path "/b652b05a-4e3d-4ad1-b032-18886abe7d45/5a98a3dd-0349-471b-8829-e40d62018b04"
-					(reference "#PWR029")
+					(reference "#PWR0102")
 					(unit 1)
 				)
@@
 		(on_board yes)
 		(dnp no)
-		(property "Reference" "C6"
+		(property "Reference" "C1"
 			(at 95.25 60.9663 0)
 			(effects
@@
 			(project "drs"
 				(path "/b652b05a-4e3d-4ad1-b032-18886abe7d45/5a98a3dd-0349-471b-8829-e40d62018b04"
-					(reference "C6")
+					(reference "C1")
 					(unit 1)
 				)
@@
 		(dnp no)
 		(fields_autoplaced yes)
-		(property "Reference" "#PWR01"
+		(property "Reference" "#PWR0104"
 			(at 156.21 142.24 0)
 			(effects
@@
 			(project "drs"
 				(path "/b652b05a-4e3d-4ad1-b032-18886abe7d45/5a98a3dd-0349-471b-8829-e40d62018b04"
-					(reference "#PWR01")
+					(reference "#PWR0104")
 					(unit 1)
 				)
@@
 		(on_board yes)
 		(dnp no)
-		(property "Reference" "C1"
+		(property "Reference" "C2"
 			(at 106.68 60.9663 0)
 			(effects
@@
 			(project "drs"
 				(path "/b652b05a-4e3d-4ad1-b032-18886abe7d45/5a98a3dd-0349-471b-8829-e40d62018b04"
-					(reference "C1")
+					(reference "C2")
 					(unit 1)
 				)
@@
 		(dnp no)
 		(fields_autoplaced yes)
-		(property "Reference" "R4"
+		(property "Reference" "R2"
 			(at 114.3 78.74 90)
 			(effects
@@
 			(project "drs"
 				(path "/b652b05a-4e3d-4ad1-b032-18886abe7d45/5a98a3dd-0349-471b-8829-e40d62018b04"
-					(reference "R4")
+					(reference "R2")
 					(unit 1)
 				)
@@
 		(dnp no)
 		(fields_autoplaced yes)
-		(property "Reference" "#FLG07"
+		(property "Reference" "#FLG0101"
 			(at 87.63 53.975 0)
 			(effects
@@
 			(project "drs"
 				(path "/b652b05a-4e3d-4ad1-b032-18886abe7d45/5a98a3dd-0349-471b-8829-e40d62018b04"
-					(reference "#FLG07")
+					(reference "#FLG0101")
 					(unit 1)
 				)
@@
 		(dnp no)
 		(fields_autoplaced yes)
-		(property "Reference" "C2"
+		(property "Reference" "C3"
 			(at 119.38 60.9662 0)
 			(effects
@@
 			(project "drs"
 				(path "/b652b05a-4e3d-4ad1-b032-18886abe7d45/5a98a3dd-0349-471b-8829-e40d62018b04"
-					(reference "C2")
+					(reference "C3")
 					(unit 1)
 				)
@@
 		(dnp no)
 		(fields_autoplaced yes)
-		(property "Reference" "C3"
+		(property "Reference" "C4"
 			(at 132.08 60.9662 0)
 			(effects
@@
 			(project "drs"
 				(path "/b652b05a-4e3d-4ad1-b032-18886abe7d45/5a98a3dd-0349-471b-8829-e40d62018b04"
-					(reference "C3")
+					(reference "C4")
 					(unit 1)
 				)
@@
 		(on_board yes)
 		(dnp no)
-		(property "Reference" "C4"
+		(property "Reference" "C5"
 			(at 144.78 60.9663 0)
 			(effects
@@
 			(project "drs"
 				(path "/b652b05a-4e3d-4ad1-b032-18886abe7d45/5a98a3dd-0349-471b-8829-e40d62018b04"
-					(reference "C4")
+					(reference "C5")
 					(unit 1)
 				)
@@
 		(dnp no)
 		(fields_autoplaced yes)
-		(property "Reference" "#PWR03"
+		(property "Reference" "#PWR0103"
 			(at 142.24 76.2 0)
 			(effects
@@
 			(project "drs"
 				(path "/b652b05a-4e3d-4ad1-b032-18886abe7d45/5a98a3dd-0349-471b-8829-e40d62018b04"
-					(reference "#PWR03")
+					(reference "#PWR0103")
 					(unit 1)
 				)
@@
 		(dnp no)
 		(fields_autoplaced yes)
-		(property "Reference" "#PWR02"
+		(property "Reference" "#PWR0101"
 			(at 107.95 85.09 0)
 			(effects
@@
 			(project "drs"
 				(path "/b652b05a-4e3d-4ad1-b032-18886abe7d45/5a98a3dd-0349-471b-8829-e40d62018b04"
-					(reference "#PWR02")
+					(reference "#PWR0101")
 					(unit 1)
 				)

Commit message: schematic & pcb update
Parts:
- added D1: LED_WRN, LED_SMD:LED_0603_1608Metric, symbol Device:LED_Small
- added D2: LED_OK, LED_SMD:LED_0603_1608Metric, symbol Device:LED_Small
- added D3: LED_ERR, LED_SMD:LED_0603_1608Metric, symbol Device:LED_Small
- added R2, R3, R4: 1k, Resistor_SMD:R_0603_1608Metric_Pad0.98x0.95mm_HandSolder, symbol Device:R_Small
- renumbered R2 to R5
Connections:
- net +3V3: now also R2.1, R3.1, R4.2
- net LED_ERR: now also D3.1 (K)
- net LED_OK: now also D2.1 (K)
- net LED_WRN: now also D1.1 (K)
- new net DERR_to_R1k: D3.2 (A), R4.1
- new net DOK_to_R1k: D2.2 (A), R3.2
- new net DWRN_to_R1k: D1.2 (A), R2.2
Other:
- moved on the sheet: C1, C2, C3, C4, C5, R1, R5, U1
