File: hardware/control.kicad_sch (KiCad schematic)
At the start: 14 parts, among them U1 STM32G0C1KCTxN

Commit message: pcb & footprint update
Parts:
- C2, C4: Mouser Price/Stock https://www.mouser.pl/ProductDetail/KEMET/C0603C104J5RACTM?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 -> https://www.mouser.pl/ProductDetail/Murata-Electronics/GRM0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
- C3, C5: footprint Capacitor_SMD:C_0603_1608Metric_Pad1.08x0.95mm_HandSolder -> Capacitor_SMD:C_0201_0603Metric_Pad0.64x0.40mm_HandSolder; Mouser Price/Stock https://www.mouser.pl/ProductDetail/TAIYO-YUDEN/MLASG168BB5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 -> https://www.mouser.pl/ProductDetail/Murata-Electronics/GRM0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
- D1, D2, D3: footprint LED_SMD:LED_0603_1608Metric -> LED_SMD:LED_0603_1608Metric_Pad1.05x0.95mm_HandSolder

Commit message: Update
Parts:
- C3, C5: footprint Capacitor_SMD:C_0201_0603Metric_Pad0.64x0.40mm_HandSolder -> Capacitor_SMD:C_0603_1608Metric_Pad1.08x0.95mm_HandSolder; Mouser Price/Stock https://www.mouser.pl/ProductDetail/Murata-Electronics/GRM0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 -> https://www.mouser.pl/ProductDetail/Murata-Electronics/GRM1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
Connections:
- net MISO: no longer names the net of U1.10 (PA3)
- net MOSI: no longer names the net of U1.11 (PA4)
- net SCK: no longer names the net of U1.7 (PA0)
- no-connect marks 12 -> 15
Other:
- moved on the sheet: C2, C5

Commit message: psb & schematic update
Parts:
- added R20, R21: 5k1, Resistor_SMD:R_0603_1608Metric_Pad0.98x0.95mm_HandSolder, symbol Device:R_Small
Connections:
- net PWM1: now also R21.2
- net PWM2: now also R20.2
- new net +5V: R20.1, R21.1

Commit message: pcb update
Changed lines of the file:
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@@
-		)
-	)
-	(label "PWM1"
-		(at 186.69 91.44 180)
-		(effects
-			(font
-				(size 1.27 1.27)
-			)
-			(justify right bottom)
 		)
 	)
@@
 		)
 	)
-	(label "PWM2"
-		(at 186.69 93.98 180)
+	(label "PWM1"
+		(at 175.26 91.44 0)
 		(effects
 			(font
 				(size 1.27 1.27)
 			)
-			(justify right bottom)
+			(justify left bottom)
 		)
 	)
@@
 		(effects
 			(font
+				(size 1.27 1.27)
+			)
+			(justify left bottom)
+		)
+	)
+	(label "PWM2"
+		(at 175.26 93.98 0)
+		(effects
+			(font

Commit message: Added author on pcb
Other:
- company: (none) -> Author: Grzegorz Potocki
- title: (none) -> DRS - Drag Reduction System
Changed lines of the file:
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@@
 	(generator_version "9.0")
 	(paper "A4")
+	(title_block
+		(title "DRS - Drag Reduction System")
+		(date "2024-11-28")
+		(rev "${REVISION}")
+		(company "Author: Grzegorz Potocki")
+		(comment 1 "Reviewer: Jakub Drankiewicz")
+	)
 	(bus_alias "CAN"
 		(members "RXD" "TXD")
