File: hardware/drs.kicad_sch (KiCad schematic)
At the start: 0 parts

Commit message: Added author on pcb
Other:
- title: Drag Reduction System -> DRS - Drag Reduction System
Changed lines of the file:
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@@
 	(paper "A4")
 	(title_block
-		(title "Drag Reduction System")
+		(title "DRS - Drag Reduction System")
 		(date "2024-11-28")
 		(rev "${REVISION}")
 		(company "Author: Grzegorz Potocki")
-		(comment 1 "Reviewer:")
+		(comment 1 "Reviewer: Jakub Drankiewicz")
 	)
 	(text "DRS"
