File: hardware/connectors.kicad_sch (KiCad schematic)
At the start: 8 parts, among them J1 USB-C_GCT_USB4145-03-0070-C, J2 FTSH-107-01-L-D-K, J3 POWER & CAN & SPI2, J4 PWM1, J5 PWM2, T13 TP_VBUS

Commit message: schematic & pcb update
Parts:
- renumbered R12 to R15, R13 to R16, T13 to T12
Connections:
- net CAN_H: now reaches J3.6 (Pin_6)
Changed lines of the file:
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@@
+		)
+	)
+	(global_label "CAN_H"
+		(shape input)
+		(at 166.37 69.85 0)
+		(fields_autoplaced yes)
+		(effects
+			(font
+				(size 1.27 1.27)
+			)
+			(justify left)
+		)
+		(property "Intersheetrefs" "${INTERSHEET_REFS}"
+			(at 175.3424 69.85 0)
+			(effects
+				(font
+					(size 1.27 1.27)
+				)
+				(justify left)
+				(hide yes)
+			)
 		)
 	)
@@
 		(dnp no)
 		(fields_autoplaced yes)
-		(property "Reference" "#PWR0123"
+		(property "Reference" "#PWR029"
 			(at 167.64 86.36 0)
 			(effects
@@
 			(project "drs"
 				(path "/b652b05a-4e3d-4ad1-b032-18886abe7d45/f3e8ebf7-786b-493f-9dff-a3955a7183ae"
-					(reference "#PWR0123")
+					(reference "#PWR029")
 					(unit 1)
 				)
@@
 		(dnp no)
 		(fields_autoplaced yes)
-		(property "Reference" "#PWR0120"
+		(property "Reference" "#PWR032"
 			(at 233.68 67.31 0)
 			(effects
@@
 			(project "drs"
 				(path "/b652b05a-4e3d-4ad1-b032-18886abe7d45/f3e8ebf7-786b-493f-9dff-a3955a7183ae"
-					(reference "#PWR0120")
+					(reference "#PWR032")
 					(unit 1)
 				)
@@
 		(dnp no)
 		(fields_autoplaced yes)
-		(property "Reference" "#PWR0130"
+		(property "Reference" "#PWR022"
 			(at 93.98 71.12 0)
 			(effects
@@
 			(project "drs"
 				(path "/b652b05a-4e3d-4ad1-b032-18886abe7d45/f3e8ebf7-786b-493f-9dff-a3955a7183ae"
-					(reference "#PWR0130")
+					(reference "#PWR022")
 					(unit 1)
 				)
@@
 		(dnp no)
 		(fields_autoplaced yes)
-		(property "Reference" "#PWR0129"
+		(property "Reference" "#PWR021"
 			(at 74.93 54.61 0)
 			(effects
@@
 			(project "drs"
 				(path "/b652b05a-4e3d-4ad1-b032-18886abe7d45/f3e8ebf7-786b-493f-9dff-a3955a7183ae"
-					(reference "#PWR0129")
+					(reference "#PWR021")
 					(unit 1)
 				)
@@
 		(dnp no)
 		(fields_autoplaced yes)
-		(property "Reference" "#PWR0131"
+		(property "Reference" "#PWR020"
 			(at 68.58 100.33 0)
 			(effects
@@
 			(project "drs"
 				(path "/b652b05a-4e3d-4ad1-b032-18886abe7d45/f3e8ebf7-786b-493f-9dff-a3955a7183ae"
-					(reference "#PWR0131")
+					(reference "#PWR020")
 					(unit 1)
 				)
@@
 		(dnp no)
 		(fields_autoplaced yes)
-		(property "Reference" "#PWR0122"
+		(property "Reference" "#PWR023"
 			(at 134.62 133.35 0)
 			(effects
@@
 			(project "drs"
 				(path "/b652b05a-4e3d-4ad1-b032-18886abe7d45/f3e8ebf7-786b-493f-9dff-a3955a7183ae"
-					(reference "#PWR0122")
+					(reference "#PWR023")
 					(unit 1)
 				)
@@
 		(dnp no)
 		(fields_autoplaced yes)
-		(property "Reference" "R12"
+		(property "Reference" "R15"
 			(at 88.9 57.15 90)
 			(effects
@@
 			(project "drs"
 				(path "/b652b05a-4e3d-4ad1-b032-18886abe7d45/f3e8ebf7-786b-493f-9dff-a3955a7183ae"
-					(reference "R12")
+					(reference "R15")
 					(unit 1)
 				)
@@
 		(on_board yes)
 		(dnp no)
-		(property "Reference" "#PWR0127"
+		(property "Reference" "#PWR030"
 			(at 172.72 64.77 0)
 			(effects
@@
 			(project "drs"
 				(path "/b652b05a-4e3d-4ad1-b032-18886abe7d45/f3e8ebf7-786b-493f-9dff-a3955a7183ae"
-					(reference "#PWR0127")
+					(reference "#PWR030")
 					(unit 1)
 				)
@@
 		(dnp no)
 		(fields_autoplaced yes)
-		(property "Reference" "#PWR0125"
+		(property "Reference" "#PWR026"
 			(at 147.32 69.85 0)
 			(effects
@@
 			(project "drs"
 				(path "/b652b05a-4e3d-4ad1-b032-18886abe7d45/f3e8ebf7-786b-493f-9dff-a3955a7183ae"
-					(reference "#PWR0125")
+					(reference "#PWR026")
 					(unit 1)
 				)
@@
 		(dnp no)
 		(fields_autoplaced yes)
-		(property "Reference" "#PWR0118"
+		(property "Reference" "#PWR031"
 			(at 233.68 57.15 0)
 			(effects
@@
 			(project "drs"
 				(path "/b652b05a-4e3d-4ad1-b032-18886abe7d45/f3e8ebf7-786b-493f-9dff-a3955a7183ae"
-					(reference "#PWR0118")
+					(reference "#PWR031")
 					(unit 1)
 				)
@@
 		(dnp no)
 		(fields_autoplaced yes)
-		(property "Reference" "#PWR0117"
+		(property "Reference" "#PWR034"
 			(at 233.68 90.17 0)
 			(effects
@@
 			(project "drs"
 				(path "/b652b05a-4e3d-4ad1-b032-18886abe7d45/f3e8ebf7-786b-493f-9dff-a3955a7183ae"
-					(reference "#PWR0117")
+					(reference "#PWR034")
 					(unit 1)
 				)
@@
 		(dnp no)
 		(fields_autoplaced yes)
-		(property "Reference" "#PWR0128"
+		(property "Reference" "#PWR025"
 			(at 147.32 67.31 0)
 			(effects
@@
 			(project "drs"
 				(path "/b652b05a-4e3d-4ad1-b032-18886abe7d45/f3e8ebf7-786b-493f-9dff-a3955a7183ae"
-					(reference "#PWR0128")
+					(reference "#PWR025")
 					(unit 1)
 				)
@@
 		(dnp no)
 		(fields_autoplaced yes)
-		(property "Reference" "T13"
+		(property "Reference" "T12"
 			(at 76.2 55.8799 0)
 			(effects
@@
 			(project "drs"
 				(path "/b652b05a-4e3d-4ad1-b032-18886abe7d45/f3e8ebf7-786b-493f-9dff-a3955a7183ae"
-					(reference "T13")
+					(reference "T12")
 					(unit 1)
 				)
@@
 		(dnp no)
 		(fields_autoplaced yes)
-		(property "Reference" "R13"
+		(property "Reference" "R16"
 			(at 88.9 69.85 90)
 			(effects
@@
 			(project "drs"
 				(path "/b652b05a-4e3d-4ad1-b032-18886abe7d45/f3e8ebf7-786b-493f-9dff-a3955a7183ae"
-					(reference "R13")
+					(reference "R16")
 					(unit 1)
 				)
@@
 		(dnp no)
 		(fields_autoplaced yes)
-		(property "Reference" "#PWR0119"
+		(property "Reference" "#PWR033"
 			(at 233.68 78.74 0)
 			(effects
@@
 			(project "drs"
 				(path "/b652b05a-4e3d-4ad1-b032-18886abe7d45/f3e8ebf7-786b-493f-9dff-a3955a7183ae"
-					(reference "#PWR0119")
+					(reference "#PWR033")
 					(unit 1)
 				)
@@
 		(dnp no)
 		(fields_autoplaced yes)
-		(property "Reference" "#PWR0121"
+		(property "Reference" "#PWR024"
 			(at 142.24 125.73 0)
 			(effects
@@
 			(project "drs"
 				(path "/b652b05a-4e3d-4ad1-b032-18886abe7d45/f3e8ebf7-786b-493f-9dff-a3955a7183ae"
-					(reference "#PWR0121")
+					(reference "#PWR024")
 					(unit 1)
 				)
@@
 		(on_board yes)
 		(dnp no)
-		(property "Reference" "#PWR0126"
+		(property "Reference" "#PWR027"
 			(at 147.32 64.77 0)
 			(effects
@@
 			(project "drs"
 				(path "/b652b05a-4e3d-4ad1-b032-18886abe7d45/f3e8ebf7-786b-493f-9dff-a3955a7183ae"
-					(reference "#PWR0126")
+					(reference "#PWR027")
 					(unit 1)
 				)
@@
 		(dnp no)
 		(fields_autoplaced yes)
-		(property "Reference" "#PWR0124"
+		(property "Reference" "#PWR028"
 			(at 152.4 86.36 0)
 			(effects
@@
 			(project "drs"
 				(path "/b652b05a-4e3d-4ad1-b032-18886abe7d45/f3e8ebf7-786b-493f-9dff-a3955a7183ae"
-					(reference "#PWR0124")
-					(unit 1)
-				)
+					(reference "#PWR028")
+					(unit 1)
+				)

Commit message: usbc changed, foots for electro cap and +5 lay
Parts:
- J1: footprint SamacSys_Parts:USB4145030230C -> Connector_USB:USB_C_Receptacle_GCT_USB4110; Mouser Price/Stock https://www.mouser.pl/ProductDetail/GCT/USB4145-03-0070-C?q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 -> https://www.mouser.pl/datasheet/2/837/GCT_USB4110_Product_D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
Changed lines of the file:
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@@
 			)
 		)
-		(property "Footprint" "SamacSys_Parts:USB4145030230C"
+		(property "Footprint" "Connector_USB:USB_C_Receptacle_GCT_USB4110"
 			(at 88.9 67.31 0)
 			(effects
@@
 			)
 		)
-		(property "Mouser Price/Stock" "https://www.mouser.pl/ProductDetail/GCT/USB4145-03-0070-C?qs=vvQtp7zwQdNoT6Ti9aciDw%3D%3D&srsltid=AfmBOoq0uP6vTzB2zbnWyQUamBuKb60wxEO7ZLPCh7hQgy-ny-YsYWrG"
+		(property "Mouser Price/Stock" "https://www.mouser.pl/datasheet/2/837/GCT_USB4110_Product_Drawing___20k_cycles-3455479.pdf"
 			(at 67.31 57.15 0)
 			(effects

Commit message: pcb & footprint update
Parts:
- removed J1: USB-C_GCT_USB4145-03-0070-C, Connector_USB:USB_C_Receptacle_GCT_USB4110, symbol USB-C_GCT_USB4145-03-0070-C:USB-C_GCT_USB4145-03-0070-C
- added J1: USB_C_Receptacle_USB2.0_16P, Connector_USB:USB_C_Receptacle_GCT_USB4105-xx-A_16P_TopMnt_Horizontal, symbol Connector:USB_C_Receptacle_USB2.0_16P
Connections:
- net D+: now also J1.A6 (D+), J1.B6 (D+)
- net D-: now also J1.A7 (D-), J1.B7 (D-)
- net GND: now also J1.A1 (GND), J1.A12 (GND), J1.B1 (GND), J1.B12 (GND), J1.S1 (SHIELD)
- net USB_CC1: now also J1.A5 (CC1)
- net USB_CC2: now also J1.B5 (CC2)
- net VBUS: now also J1.A4 (VBUS), J1.A9 (VBUS), J1.B4 (VBUS), J1.B9 (VBUS)
Other:
- moved on the sheet: J2, R15, R16, T12

Commit message: pcb update
Connections:
- net +6V6S1: no longer J3.3 (Pin_3)
- net +6V6S2: no longer J3.5 (Pin_5)
- net CAN_H: now also J3.10 (Pin_10); no longer J3.6 (Pin_6)
- net CAN_L: now also J3.12 (Pin_12); no longer J3.4 (Pin_4)
- net GND: now also J3.3 (Pin_3), J3.4 (Pin_4); no longer J3.11 (Pin_11), J3.12 (Pin_12)
- net MISO: now also J3.6 (Pin_6); no longer J3.7 (Pin_7)
- net MOSI: now also J3.8 (Pin_8); no longer J3.9 (Pin_9)
- net SCK: now also J3.5 (Pin_5); no longer J3.10 (Pin_10)
- no-connect marks 8 -> 10

Commit message: pcb update
Connections:
- net CAN_H renamed CAN_P
- net CAN_L renamed CAN_N
Changed lines of the file:
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@@
 		)
 	)
-	(global_label "CAN_H"
+	(global_label "CAN_P"
 		(shape input)
 		(at 166.37 74.93 0)
@@
 		)
 		(property "Intersheetrefs" "${INTERSHEET_REFS}"
-			(at 175.3424 74.93 0)
+			(at 175.2819 74.93 0)
 			(effects
 				(font
@@
 		)
 	)
-	(global_label "CAN_L"
+	(global_label "CAN_N"
 		(shape input)
 		(at 166.37 77.47 0)
@@
 		)
 		(property "Intersheetrefs" "${INTERSHEET_REFS}"
-			(at 175.04 77.47 0)
+			(at 175.3424 77.47 0)
 			(effects
 				(font

Commit message: Update
Parts:
- J3: value POWER & CAN & SPI2 -> POWER & CAN
Connections:
- net MISO: no longer names the net of J3.6 (Pin_6)
- net MOSI: no longer names the net of J3.8 (Pin_8)
- net SCK: no longer names the net of J3.5 (Pin_5)
- no-connect marks 10 -> 13
Other:
- note added: "POWER & CAN"
- note added: "PROGRAMMER"
- note removed: "POWER & CAN & SPI2"
- note removed: "PROGRAMATOR"

Commit message: pcb & scheme update
Parts:
- added D10, D11: SMAJ7.0CAH, Diode_SMD:D_SMA_Handsoldering, symbol Diode:SMAJ7.0A
- added D9: PESD5V0U2BT-QR, Package_TO_SOT_SMD:SOT-23-3, symbol Power_Protection:ESDA5V3L
- added R18, R19: 1k, Resistor_SMD:R_0603_1608Metric_Pad0.98x0.95mm_HandSolder, symbol Device:R_Small
Connections:
- net +6V6S1: now also D10.1 (A1)
- net +6V6S2: now also D11.1 (A1)
- net GND: now also D10.2 (A2), D11.2 (A2), D9.3 (A)
- net PWM1: now also R19.2
- net PWM2: now also R18.2
- new net PWM1_OUT: D9.2 (K), R19.1
- new net PWM2_OUT: D9.1 (K), R18.1
Other:
- moved on the sheet: J1, J3, J4, J5, R15, R16, T12
